File: star_chiplet.kicad_sch (KiCad schematic)
At the start: 0 parts

Commit message: Add files via upload
Other:
- sheet Caravel renamed Socket Connector
Changed lines of the file:
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@@
 			(project "star_chiplet"
 				(path "/1f1d514b-67fa-4200-8a91-3df4fa362116"
-					(page "5")
+					(page "2")
 				)
 			)
@@
 			(color 0 0 0 0.0000)
 		)
-		(property "Sheetname" "Caravel"
+		(property "Sheetname" "Socket Connector"
 			(at 38.1 83.1084 0)
 			(effects
@@
 			(project "star_chiplet"
 				(path "/1f1d514b-67fa-4200-8a91-3df4fa362116"
-					(page "2")
+					(page "5")
 				)
 			)
